Commit message: real_time_factor 0.99 set

File: src/car3/urdf/car3.urdf (robot description, URDF)
Before this commit: robot car3, 25 links, 24 joints
Links:
- link wheel_lb_link: geometry collision cylinder length=0.052 radius=0.0489; visual mesh filename=package://car3/meshes/wheel_lb_link.STL
- link wheel_lf_link: geometry collision cylinder length=0.052 radius=0.0489; visual mesh filename=package://car3/meshes/wheel_lf_link.STL
- link wheel_rb_link: geometry collision cylinder length=0.052 radius=0.0489; visual mesh filename=package://car3/meshes/wheel_rb_link.STL
- link wheel_rf_link: geometry collision cylinder length=0.052 radius=0.0489; visual mesh filename=package://car3/meshes/wheel_rf_link.STL

Commit message: urdf standered

File: src/car3/urdf/car3.urdf (robot description, URDF)
Before this commit: robot car3, 25 links, 24 joints
Links:
- link laser_link: geometry collision mesh filename=package://car3/meshes/laser_link.STL; visual mesh filename=package://car3/meshes/laser_link.STL
- link wheel_lb_link: geometry collision mesh filename=package://car3/meshes/wheel_lb_link.STL; visual mesh filename=package://car3/meshes/wheel_lb_link.STL
- link wheel_lf_link: geometry collision mesh filename=package://car3/meshes/wheel_lf_link.STL; visual mesh filename=package://car3/meshes/wheel_lf_link.STL
- link wheel_rb_link: geometry collision mesh filename=package://car3/meshes/wheel_rb_link.STL; visual mesh filename=package://car3/meshes/wheel_rb_link.STL
- link wheel_rf_link: geometry collision mesh filename=package://car3/meshes/wheel_rf_link.STL; visual mesh filename=package://car3/meshes/wheel_rf_link.STL
